File: pcb/shooting-star-controller/utrinek-kontroler.sch (KiCad schematic (older format))
At the start: 8 parts, among them IC1 ATTINY841-SSU, J1 RJ45, P1 CONN_01X05, P2 CONN_01X02, P3 CONN_01X06

Commit message: Double sided pcbs
Parts:
- P3: footprint attiny841-spi:ATTINY841-SPI -> Pin_Headers:Pin_Header_Straight_2x03_Pitch2.54mm
Changed lines of the file:
@@
 F 0 "P3" H 8300 4850 50  0000 C CNN
 F 1 "CONN_01X06" V 8400 4500 50  0000 C CNN
-F 2 "attiny841-spi:ATTINY841-SPI" H 8300 4500 50  0001 C CNN
+F 2 "Pin_Headers:Pin_Header_Straight_2x03_Pitch2.54mm" H 8300 4500 50  0001 C CNN
 F 3 "" H 8300 4500 50  0000 C CNN
 	1    8300 4500
